Commit message: converted hand

File: src/viz/models/titans_hand/titans_hand.urdf (robot description, URDF)
Before this commit: robot converted_robot, 55 links, 54 joints
Links:
- removed link f_distal_thumb_virtual
- removed link f_medial_thumb2f_distal_thumb_virtual_fixed_jointbody
- link base: geometry visual mesh filename=converted_connector.stl
- link f_distal_1: geometry visual mesh filename=converted_f_distal_1.stl
- link f_distal_2: geometry visual mesh filename=converted_f_distal_2.stl
- link f_distal_3: geometry visual mesh filename=converted_f_distal_3.stl
- link f_distal_4: geometry visual mesh filename=converted_f_distal_4.stl
- link f_distal_thumb: geometry visual mesh filename=converted_f_distal_thumb.stl
- link f_joint_1: geometry visual mesh filename=converted_f_joint_1.stl
- link f_joint_2: geometry visual mesh filename=converted_f_joint_2.stl
- link f_joint_3: geometry visual mesh filename=converted_f_joint_3.stl
- link f_joint_4: geometry visual mesh filename=converted_f_joint_4.stl
- link f_medial_1: geometry visual mesh filename=converted_f_medial_1.stl
- link f_medial_2: geometry visual mesh filename=converted_f_medial_2.stl
- link f_medial_3: geometry visual mesh filename=converted_f_medial_3.stl
- link f_medial_4: geometry visual mesh filename=converted_f_medial_4.stl
- link f_medial_thumb: geometry visual mesh filename=converted_f_medial_thumb.stl
- link f_proximal_1: geometry visual mesh filename=converted_f_proximal_1.stl
- link f_proximal_2: geometry visual mesh filename=converted_f_proximal_2.stl
- link f_proximal_3: geometry visual mesh filename=converted_f_proximal_3.stl
- link f_proximal_4: geometry visual mesh filename=converted_f_proximal_4.stl
- link f_proximal_thumb: geometry visual mesh filename=converted_f_proximal_thumb.stl
- link finger_1: geometry visual mesh filename=converted_f_base_1.stl
- link finger_2: geometry visual mesh filename=converted_f_base_2.stl
- link finger_3: geometry visual mesh filename=converted_f_base_3.stl
- link finger_4: geometry visual mesh filename=converted_f_base_4.stl
- link hand: geometry visual mesh filename=converted_palm.stl
- link thumb: geometry visual mesh filename=converted_thumbHinge.stl
Joints:
- removed joint f_medial_thumb2f_distal_thumb_virtual_fixed
- removed joint f_medial_thumb2f_distal_thumb_virtual_fixed_offset
- joint revolute_distal_thumb: parent f_distal_thumb_virtual -> f_medial_thumb
