Commit message: converter upgrades

File: src/viz/models/titans_hand/urdf/titans_hand.urdf (robot description, URDF)
Before this commit: robot converted_robot, 53 links, 52 joints
Links:
- removed link revolute_base_hand_jointbody
- removed link revolute_thumb_jointbody
- removed link world2base_fixed_jointbody
- link base: geometry visual mesh filename=package://viz/models/titans_hand/urdf/converted_connector.s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
- link f_distal_1: geometry visual mesh filename=package://viz/models/titans_hand/urdf/converted_f_distal_1.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
- link f_distal_2: geometry visual mesh filename=package://viz/models/titans_hand/urdf/converted_f_distal_2.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
- link f_distal_3: geometry visual mesh filename=package://viz/models/titans_hand/urdf/converted_f_distal_3.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
- link f_distal_4: geometry visual mesh filename=package://viz/models/titans_hand/urdf/converted_f_distal_4.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
- link f_distal_thumb: geometry visual mesh filename=package://viz/models/titans_hand/urdf/converted_f_distal_th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
- link f_joint_1: geometry visual mesh filename=package://viz/models/titans_hand/urdf/converted_f_joint_1.s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
- link f_joint_2: geometry visual mesh filename=package://viz/models/titans_hand/urdf/converted_f_joint_2.s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
- link f_joint_3: geometry visual mesh filename=package://viz/models/titans_hand/urdf/converted_f_joint_3.s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
- link f_joint_4: geometry visual mesh filename=package://viz/models/titans_hand/urdf/converted_f_joint_4.s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
- link f_medial_1: geometry visual mesh filename=package://viz/models/titans_hand/urdf/converted_f_medial_1.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
- link f_medial_2: geometry visual mesh filename=package://viz/models/titans_hand/urdf/converted_f_medial_2.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
- link f_medial_3: geometry visual mesh filename=package://viz/models/titans_hand/urdf/converted_f_medial_3.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
- link f_medial_4: geometry visual mesh filename=package://viz/models/titans_hand/urdf/converted_f_medial_4.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
- link f_medial_thumb: geometry visual mesh filename=package://viz/models/titans_hand/urdf/converted_f_medial_th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
- link f_proximal_1: geometry visual mesh filename=package://viz/models/titans_hand/urdf/converted_f_proximal_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
- link f_proximal_2: geometry visual mesh filename=package://viz/models/titans_hand/urdf/converted_f_proximal_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
- link f_proximal_3: geometry visual mesh filename=package://viz/models/titans_hand/urdf/converted_f_proximal_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
- link f_proximal_4: geometry visual mesh filename=package://viz/models/titans_hand/urdf/converted_f_proximal_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
- link f_proximal_thumb: geometry visual mesh filename=package://viz/models/titans_hand/urdf/converted_f_proximal_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
- link finger_1: geometry visual mesh filename=package://viz/models/titans_hand/urdf/converted_f_base_1.stl
- link finger_2: geometry visual mesh filename=package://viz/models/titans_hand/urdf/converted_f_base_2.stl
- link finger_3: geometry visual mesh filename=package://viz/models/titans_hand/urdf/converted_f_base_3.stl
- link finger_4: geometry visual mesh filename=package://viz/models/titans_hand/urdf/converted_f_base_4.stl
- link hand: geometry visual mesh filename=package://viz/models/titans_hand/urdf/converted_palm.stl
- link thumb: geometry visual mesh filename=package://viz/models/titans_hand/urdf/converted_thumbHinge.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
Joints:
- removed joint revolute_base_hand
- removed joint revolute_base_hand_offset
- removed joint revolute_thumb_offset
- removed joint world2base_fixed
- removed joint world2base_fixed_offset
- added joint base_to_hand: type fixed, parent base, child hand, origin xyz=0 0 0 rpy=0 0 0
- added joint base_to_world: type fixed, parent world, child base, origin xyz=0 0 0 rpy=0 0 0
- joint revolute_thumb: child revolute_thumb_jointbody -> thumb

Commit message: solved  bug in xml

File: src/viz/models/titans_hand/urdf/titans_hand.urdf (robot description, URDF)
Before this commit: robot converted_robot, 50 links, 49 joints
Joints:
- removed joint base_to_hand
- removed joint base_to_world
- added joint revolute_base_hand: type revolute, parent base, child hand, origin xyz=0.0 0.0 0.0295, axis 0.0 1.0 0.0, limit lower=-1.5707 upper=1.5707 effort=100 velocity=100
- added joint revolute_base_hand_offset: type fixed, parent base, child hand, origin xyz=0.0 0.0 0.0 rpy=0.0 0.0 0.0
- added joint revolute_thumb_offset: type fixed, parent hand, child thumb, origin xyz=0.0 0.0 0.0 rpy=0.0 0.0 0.0
- added joint world2base_fixed: type fixed, parent world, child base, origin xyz=0.0 0.0 0.0 rpy=0.0 0.0 0.0

Commit message: re organized stuff

File: src/viz/models/titans_hand/urdf/titans_hand.urdf (robot description, URDF)
Before this commit: robot package://viz/models/titans_hand/urdf/converted_robot, 50 links, 51 joints
Links:
- removed link base
- removed link f_distal_1
- removed link f_distal_2
- removed link f_distal_3
- removed link f_distal_4
- removed link f_distal_thumb
- removed link f_joint_1
- removed link f_joint_2
- removed link f_joint_3
- removed link f_joint_4
- removed link f_medial_1
- removed link f_medial_2
- removed link f_medial_3
- removed link f_medial_4
- removed link f_medial_thumb
- removed link f_proximal_1
- removed link f_proximal_2
- removed link f_proximal_3
- removed link f_proximal_4
- removed link f_proximal_thumb
- removed link finger_1
- removed link finger_2
- removed link finger_3
- removed link finger_4
- removed link hand
- removed link hand2finger_1_fixed_jointbody
- removed link hand2finger_2_fixed_jointbody
- removed link hand2finger_3_fixed_jointbody
- removed link hand2finger_4_fixed_jointbody
- removed link revolute_distal_1_jointbody
- removed link revolute_distal_2_jointbody
- removed link revolute_distal_3_jointbody
- removed link revolute_distal_4_jointbody
- removed link revolute_distal_thumb_jointbody
- removed link revolute_joint_1_jointbody
- removed link revolute_joint_2_jointbody
- removed link revolute_joint_3_jointbody
- removed link revolute_joint_4_jointbody
- removed link revolute_medial_1_jointbody
- removed link revolute_medial_2_jointbody
- removed link revolute_medial_3_jointbody
- removed link revolute_medial_4_jointbody
- removed link revolute_medial_thumb_jointbody
- removed link revolute_proximal_1_jointbody
- removed link revolute_proximal_2_jointbody
- removed link revolute_proximal_3_jointbody
- removed link revolute_proximal_4_jointbody
- removed link revolute_proximal_thumb_jointbody
- removed link thumb
- added link connector_base, mass 0.07977435345832029; visual mesh filename=package://viz/models/titans_hand/urdf/converted_mesh/conver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
- added link palm, mass 0.08495943957289792; visual mesh filename=package://viz/models/titans_hand/urdf/converted_mesh/conver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
- added link wrist, mass 0.08032373127609675; visual mesh filename=package://viz/models/titans_hand/urdf/converted_mesh/conver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
- link world: mass 0.0 -> None
Joints:
- removed joint hand2finger_1_fixed
- removed joint hand2finger_1_fixed_offset
- removed joint hand2finger_2_fixed
- removed joint hand2finger_2_fixed_offset
- removed joint hand2finger_3_fixed
- removed joint hand2finger_3_fixed_offset
- removed joint hand2finger_4_fixed
- removed joint hand2finger_4_fixed_offset
- removed joint revolute_base_hand_offset
- removed joint revolute_distal_1
- removed joint revolute_distal_1_offset
- removed joint revolute_distal_2
- removed joint revolute_distal_2_offset
- removed joint revolute_distal_3
- removed joint revolute_distal_3_offset
- removed joint revolute_distal_4
- removed joint revolute_distal_4_offset
- removed joint revolute_distal_thumb
- removed joint revolute_distal_thumb_offset
- removed joint revolute_joint_1
- removed joint revolute_joint_1_offset
- removed joint revolute_joint_2
- removed joint revolute_joint_2_offset
- removed joint revolute_joint_3
- removed joint revolute_joint_3_offset
- removed joint revolute_joint_4
- removed joint revolute_joint_4_offset
- removed joint revolute_medial_1
- removed joint revolute_medial_1_offset
- removed joint revolute_medial_2
- removed joint revolute_medial_2_offset
- removed joint revolute_medial_3
- removed joint revolute_medial_3_offset
- removed joint revolute_medial_4
- removed joint revolute_medial_4_offset
- removed joint revolute_medial_thumb
- removed joint revolute_medial_thumb_offset
- removed joint revolute_proximal_1
- removed joint revolute_proximal_1_offset
- removed joint revolute_proximal_2
- removed joint revolute_proximal_2_offset
- removed joint revolute_proximal_3
- removed joint revolute_proximal_3_offset
- removed joint revolute_proximal_4
- removed joint revolute_proximal_4_offset
- removed joint revolute_proximal_thumb
- removed joint revolute_proximal_thumb_offset
- removed joint revolute_thumb
- removed joint revolute_thumb_offset
- removed joint world2base_fixed
- added joint world2connector_base: type fixed, parent world, child connector_base, origin xyz=0 0 0 rpy=0 0 0
- added joint wrist_to_palm: type fixed, parent wrist, child palm, origin xyz=0 0 0.05 rpy=0 0 0
- joint revolute_base_hand: child hand -> wrist; origin xyz=0.0 0.0 0.0295 -> xyz=0.0 -0.0388 0.03 rpy=0.0 0.0 0.0; parent base -> connector_base
