Commit message: urdf

File: src/viz/models/titans_hand/urdf/titans_hand.urdf (robot description, URDF)
Before this commit: robot converted_robot, 4 links, 3 joints
Links:
- added link index_abd_jointbody, mass 0.001
- added link index_abd_virt_jointbody, mass 0.001
- added link index_base, mass 0.00362069274308756; visual mesh filename=package://viz/models/titans_hand/urdf/converted_mesh/conver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
- added link index_dp, mass 0.0014065189005047724; visual mesh filename=package://viz/models/titans_hand/urdf/converted_mesh/conver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
- added link index_dp2index_fingertip_fixed_jointbody, mass 0.001
- added link index_dp_virt, mass 0.001
- added link index_fingertip, mass 0.0
- added link index_mp, mass 0.0036096163027472743; visual mesh filename=package://viz/models/titans_hand/urdf/converted_mesh/conver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
- added link index_mp2dp_jointbody, mass 0.001
- added link index_mp2dp_virt_jointbody, mass 0.001
- added link index_mp_virt, mass 0.001
- added link index_pp, mass 0.007546046440107924; visual mesh filename=package://viz/models/titans_hand/urdf/converted_mesh/conver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
- added link index_pp2index_pp_sens_fixed_jointbody, mass 0.001
- added link index_pp2mp_jointbody, mass 0.001
- added link index_pp2mp_virt_jointbody, mass 0.001
- added link index_pp_sens, mass 0.0
- added link index_pp_virt, mass 0.001
- added link index_um, mass 0.0020507778801623494; visual mesh filename=package://viz/models/titans_hand/urdf/converted_mesh/conver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
- added link index_um_virt, mass 0.001
- added link middle_abd_jointbody, mass 0.001
- added link middle_abd_virt_jointbody, mass 0.001
- added link middle_base, mass 0.00362069274308756; visual mesh filename=package://viz/models/titans_hand/urdf/converted_mesh/conver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
- added link middle_dp, mass 0.0014065189005047724; visual mesh filename=package://viz/models/titans_hand/urdf/converted_mesh/conver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
- added link middle_dp2middle_fingertip_fixed_jointbody, mass 0.001
- added link middle_dp_virt, mass 0.001
- added link middle_fingertip, mass 0.0
- added link middle_mp, mass 0.0036096163027472743; visual mesh filename=package://viz/models/titans_hand/urdf/converted_mesh/conver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
- added link middle_mp2dp_jointbody, mass 0.001
- added link middle_mp2dp_virt_jointbody, mass 0.001
- added link middle_mp_virt, mass 0.001
- added link middle_pp, mass 0.007546046440107924; visual mesh filename=package://viz/models/titans_hand/urdf/converted_mesh/conver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
- added link middle_pp2middle_pp_sens_fixed_jointbody, mass 0.001
- added link middle_pp2mp_jointbody, mass 0.001
- added link middle_pp2mp_virt_jointbody, mass 0.001
- added link middle_pp_sens, mass 0.0
- added link middle_pp_virt, mass 0.001
- added link middle_um, mass 0.0020507778801623494; visual mesh filename=package://viz/models/titans_hand/urdf/converted_mesh/conver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
- added link middle_um_virt, mass 0.001
- added link palm2index_base_fixed_jointbody, mass 0.001
- added link palm2middle_base_fixed_jointbody, mass 0.001
- added link palm2pinky_base_fixed_jointbody, mass 0.001
- added link palm2ring_base_fixed_jointbody, mass 0.001
- added link pinky_abd_jointbody, mass 0.001
- added link pinky_abd_virt_jointbody, mass 0.001
- added link pinky_base, mass 0.00362069274308756; visual mesh filename=package://viz/models/titans_hand/urdf/converted_mesh/conver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
- added link pinky_dp, mass 0.0014065189005047724; visual mesh filename=package://viz/models/titans_hand/urdf/converted_mesh/conver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
- added link pinky_dp2pinky_fingertip_fixed_jointbody, mass 0.001
- added link pinky_dp_virt, mass 0.001
- added link pinky_fingertip, mass 0.0
- added link pinky_mp, mass 0.0036096163027472743; visual mesh filename=package://viz/models/titans_hand/urdf/converted_mesh/conver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
- added link pinky_mp2dp_jointbody, mass 0.001
- added link pinky_mp2dp_virt_jointbody, mass 0.001
- added link pinky_mp_virt, mass 0.001
- added link pinky_pp, mass 0.007546046440107924; visual mesh filename=package://viz/models/titans_hand/urdf/converted_mesh/conver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
- added link pinky_pp2mp_jointbody, mass 0.001
- added link pinky_pp2mp_virt_jointbody, mass 0.001
- added link pinky_pp2pinky_pp_sens_fixed_jointbody, mass 0.001
- added link pinky_pp_sens, mass 0.0
- added link pinky_pp_virt, mass 0.001
- added link pinky_um, mass 0.0020507778801623494; visual mesh filename=package://viz/models/titans_hand/urdf/converted_mesh/conver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
- added link pinky_um_virt, mass 0.001
- added link revolute_base_hand_jointbody, mass 0.001
- added link ring_abd_jointbody, mass 0.001
- added link ring_abd_virt_jointbody, mass 0.001
- added link ring_base, mass 0.00362069274308756; visual mesh filename=package://viz/models/titans_hand/urdf/converted_mesh/conver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
- added link ring_dp, mass 0.0014065189005047724; visual mesh filename=package://viz/models/titans_hand/urdf/converted_mesh/conver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
- added link ring_dp2ring_fingertip_fixed_jointbody, mass 0.001
- added link ring_dp_virt, mass 0.001
- added link ring_fingertip, mass 0.0
- added link ring_mp, mass 0.0036096163027472743; visual mesh filename=package://viz/models/titans_hand/urdf/converted_mesh/conver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
- added link ring_mp2dp_jointbody, mass 0.001
- added link ring_mp2dp_virt_jointbody, mass 0.001
- added link ring_mp_virt, mass 0.001
- added link ring_pp, mass 0.007546046440107924; visual mesh filename=package://viz/models/titans_hand/urdf/converted_mesh/conver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
- added link ring_pp2mp_jointbody, mass 0.001
- added link ring_pp2mp_virt_jointbody, mass 0.001
- added link ring_pp2ring_pp_sens_fixed_jointbody, mass 0.001
- added link ring_pp_sens, mass 0.0
- added link ring_pp_virt, mass 0.001
- added link ring_um, mass 0.0020507778801623494; visual mesh filename=package://viz/models/titans_hand/urdf/converted_mesh/conver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
- added link ring_um_virt, mass 0.001
- added link root2index_pp_jointbody, mass 0.001
- added link root2index_pp_virt_jointbody, mass 0.001
- added link root2middle_pp_jointbody, mass 0.001
- added link root2middle_pp_virt_jointbody, mass 0.001
- added link root2pinky_pp_jointbody, mass 0.001
- added link root2pinky_pp_virt_jointbody, mass 0.001
- added link root2ring_pp_jointbody, mass 0.001
- added link root2ring_pp_virt_jointbody, mass 0.001
- added link thumb_base, mass 0.011927349600745834; visual mesh filename=package://viz/models/titans_hand/urdf/converted_mesh/conver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
- added link thumb_base2pp_jointbody, mass 0.001
- added link thumb_dp, mass 0.0014065189510415494; visual mesh filename=package://viz/models/titans_hand/urdf/converted_mesh/conver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
- added link thumb_dp2thumb_fingertip_fixed_jointbody, mass 0.001
- added link thumb_dp_virt, mass 0.001
- added link thumb_fingertip, mass 0.0
- added link thumb_hinge_jointbody, mass 0.001
- added link thumb_mp, mass 0.0036257578156079634; visual mesh filename=package://viz/models/titans_hand/urdf/converted_mesh/conver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
- added link thumb_mp2dp_jointbody, mass 0.001
- added link thumb_mp2dp_virt_jointbody, mass 0.001
- added link thumb_mp_virt, mass 0.001
- added link thumb_pp, mass 0.008517951004271104; visual mesh filename=package://viz/models/titans_hand/urdf/converted_mesh/conver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
- added link thumb_pp2mp_jointbody, mass 0.001
- added link thumb_pp2mp_virt_jointbody, mass 0.001
- added link world2connector_base_fixed_jointbody, mass 0.001
- added link wrist2palm_fixed_jointbody, mass 0.001
- link world: mass None -> 0.0
Joints:
- removed joint world2connector_base
- removed joint wrist_to_palm
- added joint index_abd: type revolute, parent index_um_virt, child index_abd_jointbody, origin xyz=0.0 0.0 0.02317496 rpy=0.0 0.0 0.0, axis 0.0 1.0 0.0, limit lower=-0.264 upper=0.264 effort=100 velocity=100
- added joint index_abd_offset: type fixed, parent index_abd_jointbody, child index_um, origin xyz=-0.0 -0.0 -0.02317496 rpy=0.0 0.0 0.0
- added joint index_abd_virt: type revolute, parent index_base, child index_abd_virt_jointbody, origin xyz=0.0 0.0 0.00527505 rpy=0.0 0.0 0.0, axis 0.0 1.0 0.0, limit lower=-0.264 upper=0.264 effort=100 velocity=100
- added joint index_abd_virt_offset: type fixed, parent index_abd_virt_jointbody, child index_um_virt, origin xyz=-0.0 -0.0 -0.00527505 rpy=0.0 0.0 0.0
- added joint index_dp2index_fingertip_fixed: type fixed, parent index_dp, child index_dp2index_fingertip_fixed_jointbody, origin xyz=0.0 0.0 0.0 rpy=0.0 0.0 0.0
- added joint index_dp2index_fingertip_fixed_offset: type fixed, parent index_dp2index_fingertip_fixed_jointbody, child index_fingertip, origin xyz=-0.0 -0.0 -0.0 rpy=0.0 0.0 0.0
- added joint index_mp2dp: type revolute, parent index_dp_virt, child index_mp2dp_jointbody, origin xyz=0.0 0.0017961 0.09655649 rpy=0.0 0.0 0.0, axis 1.0 0.0 0.0, limit lower=-0.093 upper=0.682 effort=100 velocity=100
- added joint index_mp2dp_offset: type fixed, parent index_mp2dp_jointbody, child index_dp, origin xyz=-0.0 -0.0017961 -0.09655649 rpy=0.0 0.0 0.0
- added joint index_mp2dp_virt: type revolute, parent index_mp, child index_mp2dp_virt_jointbody, origin xyz=0.0 0.00263391 0.0882811 rpy=0.0 0.0 0.0, axis 1.0 0.0 0.0, limit lower=-0.093 upper=0.682 effort=100 velocity=100
- added joint index_mp2dp_virt_offset: type fixed, parent index_mp2dp_virt_jointbody, child index_dp_virt, origin xyz=-0.0 -0.00263391 -0.0882811 rpy=0.0 0.0 0.0
- added joint index_pp2index_pp_sens_fixed: type fixed, parent index_pp, child index_pp2index_pp_sens_fixed_jointbody, origin xyz=0.0 0.0 0.0 rpy=0.0 0.0 0.0
- added joint index_pp2index_pp_sens_fixed_offset: type fixed, parent index_pp2index_pp_sens_fixed_jointbody, child index_pp_sens, origin xyz=-0.0 -0.0 -0.0 rpy=0.0 0.0 0.0
- added joint index_pp2mp: type revolute, parent index_mp_virt, child index_pp2mp_jointbody, origin xyz=0.0 0.0029099 0.07130514 rpy=0.0 0.0 0.0, axis 1.0 0.0 0.0, limit lower=-0.131 upper=0.96 effort=100 velocity=100
- added joint index_pp2mp_offset: type fixed, parent index_pp2mp_jointbody, child index_mp, origin xyz=-0.0 -0.0029099 -0.07130514 rpy=0.0 0.0 0.0
- added joint index_pp2mp_virt: type revolute, parent index_pp, child index_pp2mp_virt_jointbody, origin xyz=0.0 0.00371958 0.06026209 rpy=0.0 0.0 0.0, axis 1.0 0.0 0.0, limit lower=-0.131 upper=0.96 effort=100 velocity=100
- added joint index_pp2mp_virt_offset: type fixed, parent index_pp2mp_virt_jointbody, child index_mp_virt, origin xyz=-0.0 -0.00371958 -0.06026209 rpy=0.0 0.0 0.0
- added joint middle_abd: type revolute, parent middle_um_virt, child middle_abd_jointbody, origin xyz=0.0 0.0 0.02317496 rpy=0.0 0.0 0.0, axis 0.0 1.0 0.0, limit lower=-0.264 upper=0.264 effort=100 velocity=100
- added joint middle_abd_offset: type fixed, parent middle_abd_jointbody, child middle_um, origin xyz=-0.0 -0.0 -0.02317496 rpy=0.0 0.0 0.0
- added joint middle_abd_virt: type revolute, parent middle_base, child middle_abd_virt_jointbody, origin xyz=0.0 0.0 0.00527505 rpy=0.0 0.0 0.0, axis 0.0 1.0 0.0, limit lower=-0.264 upper=0.264 effort=100 velocity=100
- added joint middle_abd_virt_offset: type fixed, parent middle_abd_virt_jointbody, child middle_um_virt, origin xyz=-0.0 -0.0 -0.00527505 rpy=0.0 0.0 0.0
- added joint middle_dp2middle_fingertip_fixed: type fixed, parent middle_dp, child middle_dp2middle_fingertip_fixed_jointbody, origin xyz=0.0 0.0 0.0 rpy=0.0 0.0 0.0
- added joint middle_dp2middle_fingertip_fixed_offset: type fixed, parent middle_dp2middle_fingertip_fixed_jointbody, child middle_fingertip, origin xyz=-0.0 -0.0 -0.0 rpy=0.0 0.0 0.0
- added joint middle_mp2dp: type revolute, parent middle_dp_virt, child middle_mp2dp_jointbody, origin xyz=0.0 0.0017961 0.09655649 rpy=0.0 0.0 0.0, axis 1.0 0.0 0.0, limit lower=-0.093 upper=0.682 effort=100 velocity=100
- added joint middle_mp2dp_offset: type fixed, parent middle_mp2dp_jointbody, child middle_dp, origin xyz=-0.0 -0.0017961 -0.09655649 rpy=0.0 0.0 0.0
- added joint middle_mp2dp_virt: type revolute, parent middle_mp, child middle_mp2dp_virt_jointbody, origin xyz=0.0 0.00263391 0.0882811 rpy=0.0 0.0 0.0, axis 1.0 0.0 0.0, limit lower=-0.093 upper=0.682 effort=100 velocity=100
- added joint middle_mp2dp_virt_offset: type fixed, parent middle_mp2dp_virt_jointbody, child middle_dp_virt, origin xyz=-0.0 -0.00263391 -0.0882811 rpy=0.0 0.0 0.0
- added joint middle_pp2middle_pp_sens_fixed: type fixed, parent middle_pp, child middle_pp2middle_pp_sens_fixed_jointbody, origin xyz=0.0 0.0 0.0 rpy=0.0 0.0 0.0
- added joint middle_pp2middle_pp_sens_fixed_offset: type fixed, parent middle_pp2middle_pp_sens_fixed_jointbody, child middle_pp_sens, origin xyz=-0.0 -0.0 -0.0 rpy=0.0 0.0 0.0
- added joint middle_pp2mp: type revolute, parent middle_mp_virt, child middle_pp2mp_jointbody, origin xyz=0.0 0.0029099 0.07130514 rpy=0.0 0.0 0.0, axis 1.0 0.0 0.0, limit lower=-0.131 upper=0.96 effort=100 velocity=100
- added joint middle_pp2mp_offset: type fixed, parent middle_pp2mp_jointbody, child middle_mp, origin xyz=-0.0 -0.0029099 -0.07130514 rpy=0.0 0.0 0.0
- added joint middle_pp2mp_virt: type revolute, parent middle_pp, child middle_pp2mp_virt_jointbody, origin xyz=0.0 0.00371958 0.06026209 rpy=0.0 0.0 0.0, axis 1.0 0.0 0.0, limit lower=-0.131 upper=0.96 effort=100 velocity=100
- added joint middle_pp2mp_virt_offset: type fixed, parent middle_pp2mp_virt_jointbody, child middle_mp_virt, origin xyz=-0.0 -0.00371958 -0.06026209 rpy=0.0 0.0 0.0
- added joint palm2index_base_fixed: type fixed, parent palm, child palm2index_base_fixed_jointbody, origin xyz=0.002 0.04096 0.118 rpy=0.0 0.0 1.57
- added joint palm2index_base_fixed_offset: type fixed, parent palm2index_base_fixed_jointbody, child index_base, origin xyz=-0.0 -0.0 -0.0 rpy=0.0 0.0 0.0
- added joint palm2middle_base_fixed: type fixed, parent palm, child palm2middle_base_fixed_jointbody, origin xyz=0.002 0.02163081458 0.115168462 rpy=0.00014041394505603932 -0.17453294409230335 1.5699877153702502
- added joint palm2middle_base_fixed_offset: type fixed, parent palm2middle_base_fixed_jointbody, child middle_base, origin xyz=-0.0 -0.0 -0.0 rpy=0.0 0.0 0.0
- added joint palm2pinky_base_fixed: type fixed, parent palm, child palm2pinky_base_fixed_jointbody, origin xyz=0.002 -0.01537994548 0.103767481 rpy=0.0003713332265421476 -0.43633216514869133 1.5699176774335144
- added joint palm2pinky_base_fixed_offset: type fixed, parent palm2pinky_base_fixed_jointbody, child pinky_base, origin xyz=-0.0 -0.0 -0.0 rpy=0.0 0.0 0.0
- added joint palm2ring_base_fixed: type fixed, parent palm, child palm2ring_base_fixed_jointbody, origin xyz=0.002 0.002691840889 0.1112506719 rpy=0.0002898392113429571 -0.34906573499662796 1.5699488935438706
- added joint palm2ring_base_fixed_offset: type fixed, parent palm2ring_base_fixed_jointbody, child ring_base, origin xyz=-0.0 -0.0 -0.0 rpy=0.0 0.0 0.0
- added joint pinky_abd: type revolute, parent pinky_um_virt, child pinky_abd_jointbody, origin xyz=0.0 0.0 0.02317496 rpy=0.0 0.0 0.0, axis 0.0 1.0 0.0, limit lower=-0.264 upper=0.264 effort=100 velocity=100
- added joint pinky_abd_offset: type fixed, parent pinky_abd_jointbody, child pinky_um, origin xyz=-0.0 -0.0 -0.02317496 rpy=0.0 0.0 0.0
- added joint pinky_abd_virt: type revolute, parent pinky_base, child pinky_abd_virt_jointbody, origin xyz=0.0 0.0 0.00527505 rpy=0.0 0.0 0.0, axis 0.0 1.0 0.0, limit lower=-0.264 upper=0.264 effort=100 velocity=100
- added joint pinky_abd_virt_offset: type fixed, parent pinky_abd_virt_jointbody, child pinky_um_virt, origin xyz=-0.0 -0.0 -0.00527505 rpy=0.0 0.0 0.0
- added joint pinky_dp2pinky_fingertip_fixed: type fixed, parent pinky_dp, child pinky_dp2pinky_fingertip_fixed_jointbody, origin xyz=0.0 0.0 0.0 rpy=0.0 0.0 0.0
- added joint pinky_dp2pinky_fingertip_fixed_offset: type fixed, parent pinky_dp2pinky_fingertip_fixed_jointbody, child pinky_fingertip, origin xyz=-0.0 -0.0 -0.0 rpy=0.0 0.0 0.0
- added joint pinky_mp2dp: type revolute, parent pinky_dp_virt, child pinky_mp2dp_jointbody, origin xyz=0.0 0.0017961 0.09655649 rpy=0.0 0.0 0.0, axis 1.0 0.0 0.0, limit lower=-0.093 upper=0.682 effort=100 velocity=100
- added joint pinky_mp2dp_offset: type fixed, parent pinky_mp2dp_jointbody, child pinky_dp, origin xyz=-0.0 -0.0017961 -0.09655649 rpy=0.0 0.0 0.0
- added joint pinky_mp2dp_virt: type revolute, parent pinky_mp, child pinky_mp2dp_virt_jointbody, origin xyz=0.0 0.00263391 0.0882811 rpy=0.0 0.0 0.0, axis 1.0 0.0 0.0, limit lower=-0.093 upper=0.682 effort=100 velocity=100
- added joint pinky_mp2dp_virt_offset: type fixed, parent pinky_mp2dp_virt_jointbody, child pinky_dp_virt, origin xyz=-0.0 -0.00263391 -0.0882811 rpy=0.0 0.0 0.0
- added joint pinky_pp2mp: type revolute, parent pinky_mp_virt, child pinky_pp2mp_jointbody, origin xyz=0.0 0.0029099 0.07130514 rpy=0.0 0.0 0.0, axis 1.0 0.0 0.0, limit lower=-0.131 upper=0.96 effort=100 velocity=100
- added joint pinky_pp2mp_offset: type fixed, parent pinky_pp2mp_jointbody, child pinky_mp, origin xyz=-0.0 -0.0029099 -0.07130514 rpy=0.0 0.0 0.0
- added joint pinky_pp2mp_virt: type revolute, parent pinky_pp, child pinky_pp2mp_virt_jointbody, origin xyz=0.0 0.00371958 0.06026209 rpy=0.0 0.0 0.0, axis 1.0 0.0 0.0, limit lower=-0.131 upper=0.96 effort=100 velocity=100
- added joint pinky_pp2mp_virt_offset: type fixed, parent pinky_pp2mp_virt_jointbody, child pinky_mp_virt, origin xyz=-0.0 -0.00371958 -0.06026209 rpy=0.0 0.0 0.0
- added joint pinky_pp2pinky_pp_sens_fixed: type fixed, parent pinky_pp, child pinky_pp2pinky_pp_sens_fixed_jointbody, origin xyz=0.0 0.0 0.0 rpy=0.0 0.0 0.0
- added joint pinky_pp2pinky_pp_sens_fixed_offset: type fixed, parent pinky_pp2pinky_pp_sens_fixed_jointbody, child pinky_pp_sens, origin xyz=-0.0 -0.0 -0.0 rpy=0.0 0.0 0.0
- added joint revolute_base_hand_offset: type fixed, parent revolute_base_hand_jointbody, child wrist, origin xyz=-0.0 0.0388 -0.03 rpy=0.0 0.0 0.0
- added joint ring_abd: type revolute, parent ring_um_virt, child ring_abd_jointbody, origin xyz=0.0 0.0 0.02317496 rpy=0.0 0.0 0.0, axis 0.0 1.0 0.0, limit lower=-0.264 upper=0.264 effort=100 velocity=100
- added joint ring_abd_offset: type fixed, parent ring_abd_jointbody, child ring_um, origin xyz=-0.0 -0.0 -0.02317496 rpy=0.0 0.0 0.0
- added joint ring_abd_virt: type revolute, parent ring_base, child ring_abd_virt_jointbody, origin xyz=0.0 0.0 0.00527505 rpy=0.0 0.0 0.0, axis 0.0 1.0 0.0, limit lower=-0.264 upper=0.264 effort=100 velocity=100
- added joint ring_abd_virt_offset: type fixed, parent ring_abd_virt_jointbody, child ring_um_virt, origin xyz=-0.0 -0.0 -0.00527505 rpy=0.0 0.0 0.0
- added joint ring_dp2ring_fingertip_fixed: type fixed, parent ring_dp, child ring_dp2ring_fingertip_fixed_jointbody, origin xyz=0.0 0.0 0.0 rpy=0.0 0.0 0.0
- added joint ring_dp2ring_fingertip_fixed_offset: type fixed, parent ring_dp2ring_fingertip_fixed_jointbody, child ring_fingertip, origin xyz=-0.0 -0.0 -0.0 rpy=0.0 0.0 0.0
- added joint ring_mp2dp: type revolute, parent ring_dp_virt, child ring_mp2dp_jointbody, origin xyz=0.0 0.0017961 0.09655649 rpy=0.0 0.0 0.0, axis 1.0 0.0 0.0, limit lower=-0.093 upper=0.682 effort=100 velocity=100
- added joint ring_mp2dp_offset: type fixed, parent ring_mp2dp_jointbody, child ring_dp, origin xyz=-0.0 -0.0017961 -0.09655649 rpy=0.0 0.0 0.0
- added joint ring_mp2dp_virt: type revolute, parent ring_mp, child ring_mp2dp_virt_jointbody, origin xyz=0.0 0.00263391 0.0882811 rpy=0.0 0.0 0.0, axis 1.0 0.0 0.0, limit lower=-0.093 upper=0.682 effort=100 velocity=100
- added joint ring_mp2dp_virt_offset: type fixed, parent ring_mp2dp_virt_jointbody, child ring_dp_virt, origin xyz=-0.0 -0.00263391 -0.0882811 rpy=0.0 0.0 0.0
- added joint ring_pp2mp: type revolute, parent ring_mp_virt, child ring_pp2mp_jointbody, origin xyz=0.0 0.0029099 0.07130514 rpy=0.0 0.0 0.0, axis 1.0 0.0 0.0, limit lower=-0.131 upper=0.96 effort=100 velocity=100
- added joint ring_pp2mp_offset: type fixed, parent ring_pp2mp_jointbody, child ring_mp, origin xyz=-0.0 -0.0029099 -0.07130514 rpy=0.0 0.0 0.0
- added joint ring_pp2mp_virt: type revolute, parent ring_pp, child ring_pp2mp_virt_jointbody, origin xyz=0.0 0.00371958 0.06026209 rpy=0.0 0.0 0.0, axis 1.0 0.0 0.0, limit lower=-0.131 upper=0.96 effort=100 velocity=100
- added joint ring_pp2mp_virt_offset: type fixed, parent ring_pp2mp_virt_jointbody, child ring_mp_virt, origin xyz=-0.0 -0.00371958 -0.06026209 rpy=0.0 0.0 0.0
- added joint ring_pp2ring_pp_sens_fixed: type fixed, parent ring_pp, child ring_pp2ring_pp_sens_fixed_jointbody, origin xyz=0.0 0.0 0.0 rpy=0.0 0.0 0.0
- added joint ring_pp2ring_pp_sens_fixed_offset: type fixed, parent ring_pp2ring_pp_sens_fixed_jointbody, child ring_pp_sens, origin xyz=-0.0 -0.0 -0.0 rpy=0.0 0.0 0.0
- added joint root2index_pp: type revolute, parent index_pp_virt, child root2index_pp_jointbody, origin xyz=0.0 0.00314317 0.03414407 rpy=0.0 0.0 0.0, axis 1.0 0.0 0.0, limit lower=-0.157 upper=0.829 effort=100 velocity=100
- added joint root2index_pp_offset: type fixed, parent root2index_pp_jointbody, child index_pp, origin xyz=-0.0 -0.00314317 -0.03414407 rpy=0.0 0.0 0.0
- added joint root2index_pp_virt: type revolute, parent index_um, child root2index_pp_virt_jointbody, origin xyz=0.0 0.0033 0.01691888 rpy=0.0 0.0 0.0, axis 1.0 0.0 0.0, limit lower=-0.157 upper=0.829 effort=100 velocity=100
- added joint root2index_pp_virt_offset: type fixed, parent root2index_pp_virt_jointbody, child index_pp_virt, origin xyz=-0.0 -0.0033 -0.01691888 rpy=0.0 0.0 0.0
- added joint root2middle_pp: type revolute, parent middle_pp_virt, child root2middle_pp_jointbody, origin xyz=0.0 0.00314317 0.03414407 rpy=0.0 0.0 0.0, axis 1.0 0.0 0.0, limit lower=-0.157 upper=0.829 effort=100 velocity=100
- added joint root2middle_pp_offset: type fixed, parent root2middle_pp_jointbody, child middle_pp, origin xyz=-0.0 -0.00314317 -0.03414407 rpy=0.0 0.0 0.0
- added joint root2middle_pp_virt: type revolute, parent middle_um, child root2middle_pp_virt_jointbody, origin xyz=0.0 0.0033 0.01691888 rpy=0.0 0.0 0.0, axis 1.0 0.0 0.0, limit lower=-0.157 upper=0.829 effort=100 velocity=100
- added joint root2middle_pp_virt_offset: type fixed, parent root2middle_pp_virt_jointbody, child middle_pp_virt, origin xyz=-0.0 -0.0033 -0.01691888 rpy=0.0 0.0 0.0
- added joint root2pinky_pp: type revolute, parent pinky_pp_virt, child root2pinky_pp_jointbody, origin xyz=0.0 0.00314317 0.03414407 rpy=0.0 0.0 0.0, axis 1.0 0.0 0.0, limit lower=-0.157 upper=0.829 effort=100 velocity=100
- added joint root2pinky_pp_offset: type fixed, parent root2pinky_pp_jointbody, child pinky_pp, origin xyz=-0.0 -0.00314317 -0.03414407 rpy=0.0 0.0 0.0
- added joint root2pinky_pp_virt: type revolute, parent pinky_um, child root2pinky_pp_virt_jointbody, origin xyz=0.0 0.0033 0.01691888 rpy=0.0 0.0 0.0, axis 1.0 0.0 0.0, limit lower=-0.157 upper=0.829 effort=100 velocity=100
- added joint root2pinky_pp_virt_offset: type fixed, parent root2pinky_pp_virt_jointbody, child pinky_pp_virt, origin xyz=-0.0 -0.0033 -0.01691888 rpy=0.0 0.0 0.0
- added joint root2ring_pp: type revolute, parent ring_pp_virt, child root2ring_pp_jointbody, origin xyz=0.0 0.00314317 0.03414407 rpy=0.0 0.0 0.0, axis 1.0 0.0 0.0, limit lower=-0.157 upper=0.829 effort=100 velocity=100
- added joint root2ring_pp_offset: type fixed, parent root2ring_pp_jointbody, child ring_pp, origin xyz=-0.0 -0.00314317 -0.03414407 rpy=0.0 0.0 0.0
- added joint root2ring_pp_virt: type revolute, parent ring_um, child root2ring_pp_virt_jointbody, origin xyz=0.0 0.0033 0.01691888 rpy=0.0 0.0 0.0, axis 1.0 0.0 0.0, limit lower=-0.157 upper=0.829 effort=100 velocity=100
- added joint root2ring_pp_virt_offset: type fixed, parent root2ring_pp_virt_jointbody, child ring_pp_virt, origin xyz=-0.0 -0.0033 -0.01691888 rpy=0.0 0.0 0.0
- added joint thumb_base2pp: type revolute, parent thumb_base, child thumb_base2pp_jointbody, origin xyz=0.0 0.06283 0.07774 rpy=0.0 0.0 0.0, axis 1.0 0.0 0.0, limit lower=-3.141592 upper=0.0 effort=100 velocity=100
- added joint thumb_base2pp_offset: type fixed, parent thumb_base2pp_jointbody, child thumb_pp, origin xyz=-0.0 -0.06283 -0.07774 rpy=0.0 0.0 0.0
- added joint thumb_dp2thumb_fingertip_fixed: type fixed, parent thumb_dp, child thumb_dp2thumb_fingertip_fixed_jointbody, origin xyz=0.0 0.0 0.0 rpy=0.0 0.0 0.0
- added joint thumb_dp2thumb_fingertip_fixed_offset: type fixed, parent thumb_dp2thumb_fingertip_fixed_jointbody, child thumb_fingertip, origin xyz=-0.0 -0.0 -0.0 rpy=0.0 0.0 0.0
- added joint thumb_hinge: type revolute, parent palm, child thumb_hinge_jointbody, origin xyz=0.0 0.0393 0.06872 rpy=0.0 0.0 0.0, axis 0.0 0.3420201432984737 0.9396926207958065, limit lower=-1.75 upper=0.786 effort=100 velocity=100
- added joint thumb_hinge_offset: type fixed, parent thumb_hinge_jointbody, child thumb_base, origin xyz=-0.0 -0.0393 -0.06872 rpy=0.0 0.0 0.0
- added joint thumb_mp2dp: type revolute, parent thumb_dp_virt, child thumb_mp2dp_jointbody, origin xyz=-0.00464 0.0664 0.14872 rpy=0.0 0.0 0.0, axis 0.0 1.0 0.0, limit lower=-0.093 upper=0.682 effort=100 velocity=100
- added joint thumb_mp2dp_offset: type fixed, parent thumb_mp2dp_jointbody, child thumb_dp, origin xyz=0.00464 -0.0664 -0.14872 rpy=0.0 0.0 0.0
- added joint thumb_mp2dp_virt: type revolute, parent thumb_mp, child thumb_mp2dp_virt_jointbody, origin xyz=-0.00586 0.06578 0.14053 rpy=0.0 0.0 0.0, axis 0.0 1.0 0.0, limit lower=-0.093 upper=0.682 effort=100 velocity=100
- added joint thumb_mp2dp_virt_offset: type fixed, parent thumb_mp2dp_virt_jointbody, child thumb_dp_virt, origin xyz=0.00586 -0.06578 -0.14053 rpy=0.0 0.0 0.0
- added joint thumb_pp2mp: type revolute, parent thumb_mp_virt, child thumb_pp2mp_jointbody, origin xyz=-0.00696 0.06533 0.1236 rpy=0.0 0.0 0.0, axis 0.0 1.0 0.0, limit lower=-0.131 upper=0.96 effort=100 velocity=100
- added joint thumb_pp2mp_offset: type fixed, parent thumb_pp2mp_jointbody, child thumb_mp, origin xyz=0.00696 -0.06533 -0.1236 rpy=0.0 0.0 0.0
- added joint thumb_pp2mp_virt: type revolute, parent thumb_pp, child thumb_pp2mp_virt_jointbody, origin xyz=-0.0079 0.06483 0.11245 rpy=0.0 0.0 0.0, axis 0.0 1.0 0.0, limit lower=-0.131 upper=0.96 effort=100 velocity=100
- added joint thumb_pp2mp_virt_offset: type fixed, parent thumb_pp2mp_virt_jointbody, child thumb_mp_virt, origin xyz=0.0079 -0.06483 -0.11245 rpy=0.0 0.0 0.0
- added joint world2connector_base_fixed: type fixed, parent world, child world2connector_base_fixed_jointbody, origin xyz=0.0 0.0 0.0 rpy=0.0 0.0 0.0
- added joint world2connector_base_fixed_offset: type fixed, parent world2connector_base_fixed_jointbody, child connector_base, origin xyz=-0.0 -0.0 -0.0 rpy=0.0 0.0 0.0
- added joint wrist2palm_fixed: type fixed, parent wrist, child wrist2palm_fixed_jointbody, origin xyz=0.0 0.0 0.0 rpy=0.0 0.0 0.0
- added joint wrist2palm_fixed_offset: type fixed, parent wrist2palm_fixed_jointbody, child palm, origin xyz=-0.0 -0.0 -0.0 rpy=0.0 0.0 0.0
- joint revolute_base_hand: child wrist -> revolute_base_hand_jointbody
