Commit message: retargeting sort of working

File: src/viz/models/titans_hand/urdf/titans_hand.urdf (robot description, URDF)
Before this commit: robot converted_robot, 109 links, 108 joints
Links:
- removed link world2connector_base_fixed_jointbody
- added link world2wrist_fixed_jointbody, mass 0.001
- link connector_base: mass 0.07977435345832029 -> 0.07977435345788764
- link palm: mass 0.08495943957289792 -> 0.0847094208679248
- link thumb_base: mass 0.011927349600745834 -> 0.01192734960073518
- link wrist: mass 0.08032373127609675 -> 0.08354295839941446
Joints:
- removed joint world2connector_base_fixed
- removed joint world2connector_base_fixed_offset
- added joint world2wrist_fixed: type fixed, parent world, child world2wrist_fixed_jointbody, origin xyz=0.0 0.0 0.03 rpy=0.0 0.0 0.0
- added joint world2wrist_fixed_offset: type fixed, parent world2wrist_fixed_jointbody, child wrist, origin xyz=-0.0 -0.0 -0.0 rpy=0.0 0.0 0.0
- joint index_abd: origin xyz=0.0 0.0 0.02317496 rpy=0.0 0.0 0.0 -> xyz=0.0 0.0 0.01789991 rpy=0.0 0.0 0.0
- joint index_abd_offset: origin xyz=-0.0 -0.0 -0.02317496 rpy=0.0 0.0 0.0 -> xyz=-0.0 -0.0 -0.0 rpy=0.0 0.0 0.0
- joint index_abd_virt_offset: origin xyz=-0.0 -0.0 -0.00527505 rpy=0.0 0.0 0.0 -> xyz=-0.0 -0.0 -0.0 rpy=0.0 0.0 0.0
- joint index_dp2index_fingertip_fixed: origin xyz=0.0 0.0 0.0 rpy=0.0 0.0 0.0 -> xyz=0.0 0.0 0.01309 rpy=0.0 0.0 0.0
- joint index_mp2dp: origin xyz=0.0 0.0017961 0.09655649 rpy=0.0 0.0 0.0 -> xyz=0.0 -0.00083781 0.00827539 rpy=0.0 0.0 0.0
- joint index_mp2dp_offset: origin xyz=-0.0 -0.0017961 -0.09655649 rpy=0.0 0.0 0.0 -> xyz=-0.0 -0.0 -0.0 rpy=0.0 0.0 0.0
- joint index_mp2dp_virt: origin xyz=0.0 0.00263391 0.0882811 rpy=0.0 0.0 0.0 -> xyz=0.0 -0.00027599 0.01697596 rpy=0.0 0.0 0.0
- joint index_mp2dp_virt_offset: origin xyz=-0.0 -0.00263391 -0.0882811 rpy=0.0 0.0 0.0 -> xyz=-0.0 -0.0 -0.0 rpy=0.0 0.0 0.0
- joint index_pp2mp: origin xyz=0.0 0.0029099 0.07130514 rpy=0.0 0.0 0.0 -> xyz=0.0 -0.00080968 0.01104305 rpy=0.0 0.0 0.0
- joint index_pp2mp_offset: origin xyz=-0.0 -0.0029099 -0.07130514 rpy=0.0 0.0 0.0 -> xyz=-0.0 -0.0 -0.0 rpy=0.0 0.0 0.0
- joint index_pp2mp_virt: origin xyz=0.0 0.00371958 0.06026209 rpy=0.0 0.0 0.0 -> xyz=0.0 0.00057641 0.02611802 rpy=0.0 0.0 0.0
- joint index_pp2mp_virt_offset: origin xyz=-0.0 -0.00371958 -0.06026209 rpy=0.0 0.0 0.0 -> xyz=-0.0 -0.0 -0.0 rpy=0.0 0.0 0.0
- joint middle_abd: origin xyz=0.0 0.0 0.02317496 rpy=0.0 0.0 0.0 -> xyz=0.0 0.0 0.01789991 rpy=0.0 0.0 0.0
- joint middle_abd_offset: origin xyz=-0.0 -0.0 -0.02317496 rpy=0.0 0.0 0.0 -> xyz=-0.0 -0.0 -0.0 rpy=0.0 0.0 0.0
- joint middle_abd_virt_offset: origin xyz=-0.0 -0.0 -0.00527505 rpy=0.0 0.0 0.0 -> xyz=-0.0 -0.0 -0.0 rpy=0.0 0.0 0.0
- joint middle_dp2middle_fingertip_fixed: origin xyz=0.0 0.0 0.0 rpy=0.0 0.0 0.0 -> xyz=0.0 0.0 0.01309 rpy=0.0 0.0 0.0
- joint middle_mp2dp: origin xyz=0.0 0.0017961 0.09655649 rpy=0.0 0.0 0.0 -> xyz=0.0 -0.00083781 0.00827539 rpy=0.0 0.0 0.0
- joint middle_mp2dp_offset: origin xyz=-0.0 -0.0017961 -0.09655649 rpy=0.0 0.0 0.0 -> xyz=-0.0 -0.0 -0.0 rpy=0.0 0.0 0.0
- joint middle_mp2dp_virt: origin xyz=0.0 0.00263391 0.0882811 rpy=0.0 0.0 0.0 -> xyz=0.0 -0.00027599 0.01697596 rpy=0.0 0.0 0.0
- joint middle_mp2dp_virt_offset: origin xyz=-0.0 -0.00263391 -0.0882811 rpy=0.0 0.0 0.0 -> xyz=-0.0 -0.0 -0.0 rpy=0.0 0.0 0.0
- joint middle_pp2mp: origin xyz=0.0 0.0029099 0.07130514 rpy=0.0 0.0 0.0 -> xyz=0.0 -0.00080968 0.01104305 rpy=0.0 0.0 0.0
- joint middle_pp2mp_offset: origin xyz=-0.0 -0.0029099 -0.07130514 rpy=0.0 0.0 0.0 -> xyz=-0.0 -0.0 -0.0 rpy=0.0 0.0 0.0
- joint middle_pp2mp_virt: origin xyz=0.0 0.00371958 0.06026209 rpy=0.0 0.0 0.0 -> xyz=0.0 0.00057641 0.02611802 rpy=0.0 0.0 0.0
- joint middle_pp2mp_virt_offset: origin xyz=-0.0 -0.00371958 -0.06026209 rpy=0.0 0.0 0.0 -> xyz=-0.0 -0.0 -0.0 rpy=0.0 0.0 0.0
- joint palm2index_base_fixed: origin xyz=0.002 0.04096 0.118 rpy=0.0 0.0 1.57 -> xyz=0.04096 -0.002 0.063 rpy=0.0 0.0 0.0
- joint palm2middle_base_fixed: origin xyz=0.002 0.02163081458 0.115168462 rpy=0.00014041394505603932 -0.17453294409230335 1.5699877153702502 -> xyz=0.02163081458 -0.002 0.060168462 rpy=0.0 -0.17453300000000005 0.0
- joint palm2pinky_base_fixed: origin xyz=0.002 -0.01537994548 0.103767481 rpy=0.0003713332265421476 -0.43633216514869133 1.5699176774335144 -> xyz=-0.01537994548 -0.002 0.048767481 rpy=0.0 -0.4363323130000001 0.0
- joint palm2ring_base_fixed: origin xyz=0.002 0.002691840889 0.1112506719 rpy=0.0002898392113429571 -0.34906573499662796 1.5699488935438706 -> xyz=0.002691840889 -0.002 0.056250672 rpy=0.0 -0.34906585040000015 0.0
- joint pinky_abd: origin xyz=0.0 0.0 0.02317496 rpy=0.0 0.0 0.0 -> xyz=0.0 0.0 0.01789991 rpy=0.0 0.0 0.0
- joint pinky_abd_offset: origin xyz=-0.0 -0.0 -0.02317496 rpy=0.0 0.0 0.0 -> xyz=-0.0 -0.0 -0.0 rpy=0.0 0.0 0.0
- joint pinky_abd_virt_offset: origin xyz=-0.0 -0.0 -0.00527505 rpy=0.0 0.0 0.0 -> xyz=-0.0 -0.0 -0.0 rpy=0.0 0.0 0.0
- joint pinky_dp2pinky_fingertip_fixed: origin xyz=0.0 0.0 0.0 rpy=0.0 0.0 0.0 -> xyz=0.0 0.0 0.01309 rpy=0.0 0.0 0.0
- joint pinky_mp2dp: origin xyz=0.0 0.0017961 0.09655649 rpy=0.0 0.0 0.0 -> xyz=0.0 -0.00083781 0.00827539 rpy=0.0 0.0 0.0
- joint pinky_mp2dp_offset: origin xyz=-0.0 -0.0017961 -0.09655649 rpy=0.0 0.0 0.0 -> xyz=-0.0 -0.0 -0.0 rpy=0.0 0.0 0.0
- joint pinky_mp2dp_virt: origin xyz=0.0 0.00263391 0.0882811 rpy=0.0 0.0 0.0 -> xyz=0.0 -0.00027599 0.01697596 rpy=0.0 0.0 0.0
- joint pinky_mp2dp_virt_offset: origin xyz=-0.0 -0.00263391 -0.0882811 rpy=0.0 0.0 0.0 -> xyz=-0.0 -0.0 -0.0 rpy=0.0 0.0 0.0
- joint pinky_pp2mp: origin xyz=0.0 0.0029099 0.07130514 rpy=0.0 0.0 0.0 -> xyz=0.0 -0.00080968 0.01104305 rpy=0.0 0.0 0.0
- joint pinky_pp2mp_offset: origin xyz=-0.0 -0.0029099 -0.07130514 rpy=0.0 0.0 0.0 -> xyz=-0.0 -0.0 -0.0 rpy=0.0 0.0 0.0
- joint pinky_pp2mp_virt: origin xyz=0.0 0.00371958 0.06026209 rpy=0.0 0.0 0.0 -> xyz=0.0 0.00057641 0.02611802 rpy=0.0 0.0 0.0
- joint pinky_pp2mp_virt_offset: origin xyz=-0.0 -0.00371958 -0.06026209 rpy=0.0 0.0 0.0 -> xyz=-0.0 -0.0 -0.0 rpy=0.0 0.0 0.0
- joint revolute_base_hand: axis 0.0 1.0 0.0 -> 1.0 0.0 0.0; origin xyz=0.0 -0.0388 0.03 rpy=0.0 0.0 0.0 -> xyz=0.0 0.0 0.0 rpy=0.0 0.0 0.0; parent connector_base -> wrist
- joint revolute_base_hand_offset: child wrist -> connector_base; origin xyz=-0.0 0.0388 -0.03 rpy=0.0 0.0 0.0 -> xyz=-0.0 -0.0 -0.03 rpy=0.0 0.0 0.0
- joint ring_abd: origin xyz=0.0 0.0 0.02317496 rpy=0.0 0.0 0.0 -> xyz=0.0 0.0 0.01789991 rpy=0.0 0.0 0.0
- joint ring_abd_offset: origin xyz=-0.0 -0.0 -0.02317496 rpy=0.0 0.0 0.0 -> xyz=-0.0 -0.0 -0.0 rpy=0.0 0.0 0.0
- joint ring_abd_virt_offset: origin xyz=-0.0 -0.0 -0.00527505 rpy=0.0 0.0 0.0 -> xyz=-0.0 -0.0 -0.0 rpy=0.0 0.0 0.0
- joint ring_dp2ring_fingertip_fixed: origin xyz=0.0 0.0 0.0 rpy=0.0 0.0 0.0 -> xyz=0.0 0.0 0.01309 rpy=0.0 0.0 0.0
- joint ring_mp2dp: origin xyz=0.0 0.0017961 0.09655649 rpy=0.0 0.0 0.0 -> xyz=0.0 -0.00083781 0.00827539 rpy=0.0 0.0 0.0
- joint ring_mp2dp_offset: origin xyz=-0.0 -0.0017961 -0.09655649 rpy=0.0 0.0 0.0 -> xyz=-0.0 -0.0 -0.0 rpy=0.0 0.0 0.0
- joint ring_mp2dp_virt: origin xyz=0.0 0.00263391 0.0882811 rpy=0.0 0.0 0.0 -> xyz=0.0 -0.00027599 0.01697596 rpy=0.0 0.0 0.0
- joint ring_mp2dp_virt_offset: origin xyz=-0.0 -0.00263391 -0.0882811 rpy=0.0 0.0 0.0 -> xyz=-0.0 -0.0 -0.0 rpy=0.0 0.0 0.0
- joint ring_pp2mp: origin xyz=0.0 0.0029099 0.07130514 rpy=0.0 0.0 0.0 -> xyz=0.0 -0.00080968 0.01104305 rpy=0.0 0.0 0.0
- joint ring_pp2mp_offset: origin xyz=-0.0 -0.0029099 -0.07130514 rpy=0.0 0.0 0.0 -> xyz=-0.0 -0.0 -0.0 rpy=0.0 0.0 0.0
- joint ring_pp2mp_virt: origin xyz=0.0 0.00371958 0.06026209 rpy=0.0 0.0 0.0 -> xyz=0.0 0.00057641 0.02611802 rpy=0.0 0.0 0.0
- joint ring_pp2mp_virt_offset: origin xyz=-0.0 -0.00371958 -0.06026209 rpy=0.0 0.0 0.0 -> xyz=-0.0 -0.0 -0.0 rpy=0.0 0.0 0.0
- joint root2index_pp: origin xyz=0.0 0.00314317 0.03414407 rpy=0.0 0.0 0.0 -> xyz=0.0 -0.00015683 0.01722519 rpy=0.0 0.0 0.0
- joint root2index_pp_offset: origin xyz=-0.0 -0.00314317 -0.03414407 rpy=0.0 0.0 0.0 -> xyz=-0.0 -0.0 -0.0 rpy=0.0 0.0 0.0
- joint root2index_pp_virt: origin xyz=0.0 0.0033 0.01691888 rpy=0.0 0.0 0.0 -> xyz=0.0 0.0033 -0.00625608 rpy=0.0 0.0 0.0
- joint root2index_pp_virt_offset: origin xyz=-0.0 -0.0033 -0.01691888 rpy=0.0 0.0 0.0 -> xyz=-0.0 -0.0 -0.0 rpy=0.0 0.0 0.0
- joint root2middle_pp: origin xyz=0.0 0.00314317 0.03414407 rpy=0.0 0.0 0.0 -> xyz=0.0 -0.00015683 0.01722519 rpy=0.0 0.0 0.0
- joint root2middle_pp_offset: origin xyz=-0.0 -0.00314317 -0.03414407 rpy=0.0 0.0 0.0 -> xyz=-0.0 -0.0 -0.0 rpy=0.0 0.0 0.0
- joint root2middle_pp_virt: origin xyz=0.0 0.0033 0.01691888 rpy=0.0 0.0 0.0 -> xyz=0.0 0.0033 -0.00625608 rpy=0.0 0.0 0.0
- joint root2middle_pp_virt_offset: origin xyz=-0.0 -0.0033 -0.01691888 rpy=0.0 0.0 0.0 -> xyz=-0.0 -0.0 -0.0 rpy=0.0 0.0 0.0
- joint root2pinky_pp: origin xyz=0.0 0.00314317 0.03414407 rpy=0.0 0.0 0.0 -> xyz=0.0 -0.00015683 0.01722519 rpy=0.0 0.0 0.0
- joint root2pinky_pp_offset: origin xyz=-0.0 -0.00314317 -0.03414407 rpy=0.0 0.0 0.0 -> xyz=-0.0 -0.0 -0.0 rpy=0.0 0.0 0.0
- joint root2pinky_pp_virt: origin xyz=0.0 0.0033 0.01691888 rpy=0.0 0.0 0.0 -> xyz=0.0 0.0033 -0.00625608 rpy=0.0 0.0 0.0
- joint root2pinky_pp_virt_offset: origin xyz=-0.0 -0.0033 -0.01691888 rpy=0.0 0.0 0.0 -> xyz=-0.0 -0.0 -0.0 rpy=0.0 0.0 0.0
- joint root2ring_pp: origin xyz=0.0 0.00314317 0.03414407 rpy=0.0 0.0 0.0 -> xyz=0.0 -0.00015683 0.01722519 rpy=0.0 0.0 0.0
- joint root2ring_pp_offset: origin xyz=-0.0 -0.00314317 -0.03414407 rpy=0.0 0.0 0.0 -> xyz=-0.0 -0.0 -0.0 rpy=0.0 0.0 0.0
- joint root2ring_pp_virt: origin xyz=0.0 0.0033 0.01691888 rpy=0.0 0.0 0.0 -> xyz=0.0 0.0033 -0.00625608 rpy=0.0 0.0 0.0
- joint root2ring_pp_virt_offset: origin xyz=-0.0 -0.0033 -0.01691888 rpy=0.0 0.0 0.0 -> xyz=-0.0 -0.0 -0.0 rpy=0.0 0.0 0.0
- joint thumb_base2pp: axis 1.0 0.0 0.0 -> 0.0 1.0 0.0; limit lower=-3.141592 upper=0.0 effort=100 velocity=100 -> lower=-0.2 upper=1.35 effort=100 velocity=100; origin xyz=0.0 0.06283 0.07774 rpy=0.0 0.0 0.0 -> xyz=0.02053 0.0 0.007747733972 rpy=0.0 0.0 0.0
- joint thumb_base2pp_offset: origin xyz=-0.0 -0.06283 -0.07774 rpy=0.0 0.0 0.0 -> xyz=-0.0 -0.0 -0.0 rpy=0.0 0.0 0.0
- joint thumb_dp2thumb_fingertip_fixed: origin xyz=0.0 0.0 0.0 rpy=0.0 0.0 0.0 -> xyz=0.0 0.0 0.01465 rpy=0.0 0.0 0.0
- joint thumb_hinge: axis 0.0 0.3420201432984737 0.9396926207958065 -> 0.0 0.0 1.0; limit lower=-1.75 upper=0.786 effort=100 velocity=100 -> lower=-1.75 upper=0.1 effort=100 velocity=100; origin xyz=0.0 0.0393 0.06872 rpy=0.0 0.0 0.0 -> xyz=0.0393 0.0 0.023115 rpy=0.0 0.3490658500000001 0.0
- joint thumb_hinge_offset: origin xyz=-0.0 -0.0393 -0.06872 rpy=0.0 0.0 0.0 -> xyz=-0.0 -0.0 -0.0 rpy=0.0 0.0 0.0
- joint thumb_mp2dp: axis 0.0 1.0 0.0 -> 1.0 0.0 0.0; origin xyz=-0.00464 0.0664 0.14872 rpy=0.0 0.0 0.0 -> xyz=0.0 -0.00121 0.00845 rpy=0.0 0.0 0.0
- joint thumb_mp2dp_offset: origin xyz=0.00464 -0.0664 -0.14872 rpy=0.0 0.0 0.0 -> xyz=-0.0 -0.0 -0.0 rpy=0.0 0.0 0.0
- joint thumb_mp2dp_virt: axis 0.0 1.0 0.0 -> 1.0 0.0 0.0; origin xyz=-0.00586 0.06578 0.14053 rpy=0.0 0.0 0.0 -> xyz=0.0 -0.0011 0.01693 rpy=0.0 0.0 0.0
- joint thumb_mp2dp_virt_offset: origin xyz=0.00586 -0.06578 -0.14053 rpy=0.0 0.0 0.0 -> xyz=-0.0 -0.0 -0.0 rpy=0.0 0.0 0.0
- joint thumb_pp2mp: axis 0.0 1.0 0.0 -> 1.0 0.0 0.0; origin xyz=-0.00696 0.06533 0.1236 rpy=0.0 0.0 0.0 -> xyz=0.0 -0.00094 0.01115 rpy=0.0 0.0 0.0
- joint thumb_pp2mp_offset: origin xyz=0.00696 -0.06533 -0.1236 rpy=0.0 0.0 0.0 -> xyz=-0.0 -0.0 -0.0 rpy=0.0 0.0 0.0
- joint thumb_pp2mp_virt: axis 0.0 1.0 0.0 -> 1.0 0.0 0.0; origin xyz=-0.0079 0.06483 0.11245 rpy=0.0 0.0 0.0 -> xyz=0.0 0.0079 0.03471 rpy=0.0 0.0 0.0
- joint thumb_pp2mp_virt_offset: origin xyz=0.0079 -0.06483 -0.11245 rpy=0.0 0.0 0.0 -> xyz=-0.0 -0.0 -0.0 rpy=0.0 0.0 0.0
- joint wrist2palm_fixed: origin xyz=0.0 0.0 0.0 rpy=0.0 0.0 0.0 -> xyz=0.0 0.0 0.025 rpy=0.0 0.0 0.0

Commit message: mostly working, adding another keyvector does not solve the problem with the thumb

File: src/viz/models/titans_hand/urdf/titans_hand.urdf (robot description, URDF)
Before this commit: robot converted_robot, 109 links, 108 joints
Links:
- link palm: mass 0.0847094208679248 -> 0.0780873173122749
